Commit message: updated horti model

File: urdf/horti_robot_description.urdf (robot description, URDF)
Before this commit: robot horti, 60 links, 59 joints
Links:
- added link zed2i_link; collision mesh filename=package://horti_description/meshes/camera/zed2i.stl; visual mesh filename=package://horti_description/meshes/camera/zed2i.stl
- link arm_left_link1: geometry collision mesh filename=package://horti_description/meshes/xarm7/visual/link1.STL; visual mesh filename=package://horti_description/meshes/xarm7/visual/link1.STL
- link arm_left_link2: geometry collision mesh filename=package://horti_description/meshes/xarm7/visual/link2.STL; visual mesh filename=package://horti_description/meshes/xarm7/visual/link2.STL
- link arm_left_link3: geometry collision mesh filename=package://horti_description/meshes/xarm7/visual/link3.STL; visual mesh filename=package://horti_description/meshes/xarm7/visual/link3.STL
- link arm_left_link4: geometry collision mesh filename=package://horti_description/meshes/xarm7/visual/link4.STL; visual mesh filename=package://horti_description/meshes/xarm7/visual/link4.STL
- link arm_left_link5: geometry collision mesh filename=package://horti_description/meshes/xarm7/visual/link5.STL; visual mesh filename=package://horti_description/meshes/xarm7/visual/link5.STL
- link arm_left_link6: geometry collision mesh filename=package://horti_description/meshes/xarm7/visual/link6.STL; visual mesh filename=package://horti_description/meshes/xarm7/visual/link6.STL
- link arm_left_link7: geometry collision mesh filename=package://horti_description/meshes/xarm7/visual/link7.STL; visual mesh filename=package://horti_description/meshes/xarm7/visual/link7.STL
- link arm_left_link_base: geometry collision mesh filename=package://horti_description/meshes/xarm7/visual/link_base.S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; visual mesh filename=package://horti_description/meshes/xarm7/visual/link_base.S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
- link arm_right_gripper_link: geometry collision mesh filename=package://horti_description/meshes/gripper/4Finger_collisio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 scale=0.001 0.001 0.001; visual mesh filename=package://horti_description/meshes/gripper/4Finger_visual.s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 scale=0.001 0.001 0.001
- link arm_right_link1: geometry collision mesh filename=package://horti_description/meshes/xarm7/visual/link1.STL; visual mesh filename=package://horti_description/meshes/xarm7/visual/link1.STL
- link arm_right_link2: geometry collision mesh filename=package://horti_description/meshes/xarm7/visual/link2.STL; visual mesh filename=package://horti_description/meshes/xarm7/visual/link2.STL
- link arm_right_link3: geometry collision mesh filename=package://horti_description/meshes/xarm7/visual/link3.STL; visual mesh filename=package://horti_description/meshes/xarm7/visual/link3.STL
- link arm_right_link4: geometry collision mesh filename=package://horti_description/meshes/xarm7/visual/link4.STL; visual mesh filename=package://horti_description/meshes/xarm7/visual/link4.STL
- link arm_right_link5: geometry collision mesh filename=package://horti_description/meshes/xarm7/visual/link5.STL; visual mesh filename=package://horti_description/meshes/xarm7/visual/link5.STL
- link arm_right_link6: geometry collision mesh filename=package://horti_description/meshes/xarm7/visual/link6.STL; visual mesh filename=package://horti_description/meshes/xarm7/visual/link6.STL
- link arm_right_link7: geometry collision mesh filename=package://horti_description/meshes/xarm7/visual/link7.STL; visual mesh filename=package://horti_description/meshes/xarm7/visual/link7.STL
- link arm_right_link_base: geometry collision mesh filename=package://horti_description/meshes/xarm7/visual/link_base.S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; visual mesh filename=package://horti_description/meshes/xarm7/visual/link_base.S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
- link head_link1: geometry collision mesh filename=package://horti_description/meshes/lite6/visual/link1.stl; visual mesh filename=package://horti_description/meshes/lite6/visual/link1.stl
- link head_link2: geometry collision mesh filename=package://horti_description/meshes/lite6/visual/link2.stl; visual mesh filename=package://horti_description/meshes/lite6/visual/link2.stl
- link head_link3: geometry collision mesh filename=package://horti_description/meshes/lite6/visual/link3.stl; visual mesh filename=package://horti_description/meshes/lite6/visual/link3.stl
- link head_link4: geometry collision mesh filename=package://horti_description/meshes/lite6/visual/link4.stl; visual mesh filename=package://horti_description/meshes/lite6/visual/link4.stl
- link head_link5: geometry collision mesh filename=package://horti_description/meshes/lite6/visual/link5.stl; visual mesh filename=package://horti_description/meshes/lite6/visual/link5.stl
- link head_link6: geometry collision mesh filename=package://horti_description/meshes/lite6/visual/link6.stl; visual mesh filename=package://horti_description/meshes/lite6/visual/link6.stl
- link head_link_base: geometry collision mesh filename=package://horti_description/meshes/lite6/visual/base.stl; visual mesh filename=package://horti_description/meshes/lite6/visual/base.stl
- link head_mount_link: geometry collision mesh filename=package://horti_description/meshes/lite6/visual/xarm6LiteHo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; visual mesh filename=package://horti_description/meshes/lite6/visual/xarm6LiteHo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
- link zed2i_holder_link: geometry collision mesh filename=package://horti_description/meshes/camera/ZED2i_adaptor.STL; visual mesh filename=package://horti_description/meshes/camera/ZED2i_adaptor.STL
Joints:
- added joint zed2i_joint: type fixed, parent zed2i_holder_link, child zed2i_link, origin xyz=0 0 0.044 rpy=3.141592653589793 -1.5707963267948966 0

Commit message: updated horti model

File: urdf/horti_robot_description.urdf (robot description, URDF)
Before this commit: robot horti, 61 links, 60 joints
Links:
- link zed2i_link: geometry collision mesh filename=package://horti_description/meshes/camera/zed2i.stl
